Commit message: added global CS to urdf

File: Software/URDF_Files/URDF/src/new_arm/urdf/new_arm.urdf (robot description, URDF)
Before this commit: robot Lamp_urdf, 7 links, 6 joints
Links:
- removed link EE
- removed link Link1
- removed link Link2
- removed link Link3
- removed link Link4
- removed link Link5
- added link EE_link, mass 1.07322722870269; collision mesh filename=package://new_arm/meshes/EE_link.STL; visual mesh filename=package://new_arm/meshes/EE_link.STL
- added link link_1, mass 0.121759656689666; collision mesh filename=package://new_arm/meshes/link_1.STL; visual mesh filename=package://new_arm/meshes/link_1.STL
- added link link_2, mass 0.164059961594958; collision mesh filename=package://new_arm/meshes/link_2.STL; visual mesh filename=package://new_arm/meshes/link_2.STL
- added link link_3, mass 0.133281294923395; collision mesh filename=package://new_arm/meshes/link_3.STL; visual mesh filename=package://new_arm/meshes/link_3.STL
- added link link_4, mass 0.0616446065967099; collision mesh filename=package://new_arm/meshes/link_4.STL; visual mesh filename=package://new_arm/meshes/link_4.STL
- added link link_5, mass 0.082003985184141; collision mesh filename=package://new_arm/meshes/link_5.STL; visual mesh filename=package://new_arm/meshes/link_5.STL
- link base_link: mass 0.7864 -> 0.78639641308392; geometry collision mesh filename=package://new_arm/meshes/base_link.STL; visual mesh filename=package://new_arm/meshes/base_link.STL
Joints:
- removed joint Joint1
- removed joint Joint2
- removed joint Joint3
- removed joint Joint4
- removed joint Joint5
- removed joint Joint6
- added joint joint_1: type revolute, parent base_link, child link_1, origin xyz=0 0 0 rpy=0 0 0, axis 0 0 -1, limit lower=-3.14 upper=3.14 effort=0 velocity=0
- added joint joint_2: type revolute, parent link_1, child link_2, origin xyz=0.037707 0 0.057666 rpy=0 0 0, axis 0 1 0, limit lower=-3.14 upper=3.14 effort=0 velocity=0
- added joint joint_3: type revolute, parent link_2, child link_3, origin xyz=0 -5E-05 0.087 rpy=0 0 0, axis 0 1 0, limit lower=-3.14 upper=3.14 effort=0 velocity=0
- added joint joint_4: type revolute, parent link_3, child link_4, origin xyz=0 0 0.0712 rpy=0 0 0, axis 0 0 1, limit lower=-3.14 upper=3.14 effort=0 velocity=0
- added joint joint_5: type revolute, parent link_4, child link_5, origin xyz=0 0 0.0415 rpy=0 0 0, axis 0 1 0, limit lower=-3.14 upper=3.14 effort=0 velocity=0
- added joint joint_6: type revolute, parent link_5, child EE_link, origin xyz=0 0 0.05975 rpy=0 0 0, axis 0 0 1, limit lower=-3.14 upper=3.14 effort=0 velocity=0
